File: pcb/mainboard/motor-ctrl-mainboard.kicad_sch (KiCad schematic)
At the start: 149 parts, among them J1 PWR_12V, J10 I2C, J11 UP_STREAM, J12 UART, J14 OTEMP1, J15 OTEMP2, J2 CTRL_U, J21 PWR_BRIDGE, J3 CTRL_V, J4 CTRL_W, J5 I_SENSE_U, J6 I_SENSE_V, J7 I_SENSE_W, J8 HALL, J9 SWD, Q1 SS8050, Q2 SS8550, Q3 SS8050, U1 STM32F030K6Tx, U2 INA240A2D, U3 INA240A2D, U4 INA240A2D, U5 AMS1117-3.3, U6 LM339, U7 LM339, Y1 8MHz

Commit message: foc saved before auto-debug
Parts:
- removed C32: 470nF, Capacitor_SMD:C_0805_2012Metric_Pad1.18x1.45mm_HandSolder, symbol Device:C
- removed C34: 0.1uF, Capacitor_SMD:C_0603_1608Metric_Pad1.08x0.95mm_HandSolder, symbol Device:C
- removed C35, C37, C4: 10uF, Capacitor_SMD:C_1206_3216Metric_Pad1.33x1.80mm_HandSolder, symbol Device:C
- removed D2, D3: 1N4148, Diode_SMD:D_SOD-323_HandSoldering, symbol Diode:1N4007
- removed D9: SMAJ5.0A, Diode_SMD:D_SMA_Handsoldering, symbol Device:D_TVS
- removed J11: UP_STREAM, Connector_PinSocket_2.54mm:PinSocket_1x02_P2.54mm_Vertical, symbol Connector:Conn_01x02_Pin
- removed J2: CTRL_U, Connector_PinHeader_2.54mm:PinHeader_1x04_P2.54mm_Vertical, symbol Connector:Conn_01x04_Pin
- removed J21: PWR_BRIDGE, TerminalBlock_Phoenix:TerminalBlock_Phoenix_MKDS-1,5-2-5.08_1x02_P5.08mm_Horizontal, symbol Connector:Screw_Terminal_01x02
- removed J3: CTRL_V, Connector_PinHeader_2.54mm:PinHeader_1x04_P2.54mm_Vertical, symbol Connector:Conn_01x04_Pin
- removed J4: CTRL_W, Connector_PinHeader_2.54mm:PinHeader_1x04_P2.54mm_Vertical, symbol Connector:Conn_01x04_Pin
- removed Q1, Q3: SS8050, Package_TO_SOT_SMD:SOT-23, symbol Transistor_BJT:SS8050
- removed Q2: SS8550, Package_TO_SOT_SMD:SOT-23, symbol Transistor_BJT:SS8550
- removed R43, R44: 0R, Resistor_SMD:R_0603_1608Metric_Pad0.98x0.95mm_HandSolder, symbol Device:R
- removed TP6, TP7, TP9: TestPoint, TestPoint:TestPoint_Pad_D1.5mm, symbol Connector:TestPoint
- added C34, C35: 100uF/50V, Capacitor_THT:CP_Radial_D8.0mm_P3.50mm, symbol Device:C_Polarized_US
- added C4: 22uF/25V, Capacitor_Tantalum_SMD:CP_EIA-3528-21_Kemet-B_HandSolder, symbol Device:C_Polarized_US
- added D2: SS14, Diode_SMD:D_SMA_Handsoldering, symbol Diode:SS14
- added F2: 15A, basic_footprints:XF-506P, symbol Device:Polyfuse
- added J2: BRIDGE_PWR, TerminalBlock_Phoenix:TerminalBlock_Phoenix_MKDS-1,5-2-5.08_1x02_P5.08mm_Horizontal, symbol Connector:Screw_Terminal_01x02
- added J3: BRIDGE_CTRL, Connector_PinHeader_2.54mm:PinHeader_1x10_P2.54mm_Vertical, symbol Connector:Conn_01x10_Pin
- added L1: 10uH, Inductor_SMD:L_1008_2520Metric_Pad1.43x2.20mm_HandSolder, symbol Device:L
- added Q1: BSS138, digikey-footprints:SOT-23-3, symbol dk_Transistors-FETs-MOSFETs-Single:BSS138
- added U8: 7812, Package_TO_SOT_SMD:TO-252-2, symbol Regulator_Linear:L7812
- C10: value 0.1uF -> 1uF/50V; footprint Capacitor_SMD:C_0603_1608Metric_Pad1.08x0.95mm_HandSolder -> Capacitor_SMD:C_1206_3216Metric_Pad1.33x1.80mm_HandSolder
- C36: footprint Capacitor_SMD:C_0603_1608Metric_Pad1.08x0.95mm_HandSolder -> Capacitor_SMD:C_1206_3216Metric_Pad1.33x1.80mm_HandSolder
- C38: value 10uF -> 0.1uF
- D6: value SS34 -> SS14; footprint Diode_SMD:D_SMB_Handsoldering -> Diode_SMD:D_SMA_Handsoldering
- D7: value SMBJ14A -> SMBJ26A
- F1: value 2A -> 500mA; footprint Fuse:Fuse_1812_4532Metric_Pad1.30x3.40mm_HandSolder -> Fuse:Fuse_1206_3216Metric_Pad1.42x1.75mm_HandSolder
- H4: now fitted
- J1: value PWR_12V -> PWR_24V
- R24: value 10k -> 12k
- R25: value 2.2k -> 220R
- R28: value 470R -> 100k; footprint Resistor_SMD:R_2010_5025Metric_Pad1.40x2.65mm_HandSolder -> Resistor_SMD:R_0603_1608Metric_Pad0.98x0.95mm_HandSolder
- R30: value 39k -> 18k
- R31: value 10k -> 1k
- renumbered J8 to J4, J9 to J8, J12 to J9
Connections:
- net +12V: now also U8.3 (OUT); no longer C36.1, D6.1 (K), R28.1, R30.1
- net +3V3: now also C4.1; no longer C10.1
- net GND: now also R28.1, C34.2, C35.2, C4.2, J2.1 (Pin_1), J3.2 (Pin_2), J3.5 (Pin_5), J3.8 (Pin_8), Q1.2 (S), U8.2 (GND)
- net PWM_U_H: now also J3.4 (Pin_4)
- net PWM_U_L: now also J3.3 (Pin_3)
- net PWM_V_H: now also J3.7 (Pin_7)
- net PWM_V_L: now also J3.6 (Pin_6)
- net PWM_W_H: now also J3.10 (Pin_10)
- net PWM_W_L: now also J3.9 (Pin_9)
- net V_BOOST: now also C34.1, D2.1 (K), J3.1 (Pin_1)
- net +24V_RAW: now reaches F1.1, J1.2 (Pin_2)
- net +24V_RAW: now also D7.1 (A1), F2.2
- net at D6.2 (A), F1.2: no longer D7.1 (A1)
- net at R25.2: now also R28.2, Q1.1 (G)
- new net: D2.2 (A), L1.2, Q1.3 (D)
- new net: F2.1, J2.2 (Pin_2)
- new net +24V: C10.1, C35.1, C36.1, D6.1 (K), L1.1, R30.1, U8.1 (IN)
Other:
- moved on the sheet: C1, C27, C38, D1, D4, D7, D8, FB1, J10, J8, J9, R24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
